Commit message: refactor: update robot TF chain by configuring base_footprint to base_link static transform and adding joint_state_publisher

File: urdf/amr_robot.urdf.xacro (robot description, xacro)
@@ -1,21 +1,27 @@
 <?xml version="1.0"?>
 <robot name="amr_robot" xmlns:xacro="http://www.ros.org/wiki/xacro">
+  <xacro:property name="base_l"     value="0.265"/>
+  <xacro:property name="base_w"     value="0.265"/>
+  <xacro:property name="base_h"     value="0.130"/>
+  <xacro:property name="base_mass"  value="10.0"/>
+  <xacro:property name="wheel_r"    value="0.0425"/>
+  <xacro:property name="wheel_t"    value="0.018"/>
+  <xacro:property name="wheel_mass" value="0.5"/>
+  <xacro:property name="wheel_sep"  value="0.28"/>
+  <xacro:property name="caster_r"   value="0.015"/>
   <!-- ═══════════════════════════════════════════════
-       LINOROBOT2 2WD DIMENSIONS
-       base_link is the ROOT — no dummy base_footprint
-       base_footprint published via static TF in launch
+       TF CHAIN:
+       odom → base_footprint → base_link → sensors
+       base_footprint: on the ground (z=0)
+       base_link: center at wheel_r above ground
+       wheel joints: at z=0 relative to base_link
+         (wheel axle = base_link center = wheel_r above ground)
        ═══════════════════════════════════════════════ -->
-  <xacro:property name="base_l"      value="0.265"/>
-  <xacro:property name="base_w"      value="0.265"/>
-  <xacro:property name="base_h"      value="0.130"/>
-  <xacro:property name="base_mass"   value="10.0"/>
-  <xacro:property name="wheel_r"     value="0.0425"/>
-  <xacro:property name="wheel_t"     value="0.018"/>
-  <xacro:property name="wheel_mass"  value="0.5"/>
-  <xacro:property name="wheel_sep"   value="0.28"/>
-  <xacro:property name="caster_r"    value="0.015"/>
-  <!-- ═══════════════════════════════════════════════
-       BASE LINK — root link, has mass and inertia
-       ═══════════════════════════════════════════════ -->
+  <!-- <link name="base_footprint"/>
+  <joint name="base_footprint_joint" type="fixed">
+    <parent link="base_footprint"/>
+    <child  link="base_link"/>
+    <origin xyz="0 0 ${wheel_r}" rpy="0 0 0"/>
+  </joint> -->
   <link name="base_link">
     <visual>
@@ -45,7 +51,4 @@
     </inertial>
   </link>
-  <!-- ═══════════════════════════════════════════════
-       TOP DECK
-       ═══════════════════════════════════════════════ -->
   <link name="top_deck">
     <visual>
@@ -73,7 +76,4 @@
     <origin xyz="0 0 ${base_h/2+0.003}" rpy="0 0 0"/>
   </joint>
-  <!-- ═══════════════════════════════════════════════
-       ARM MOUNT — Phase 3 arm bolts here
-       ═══════════════════════════════════════════════ -->
   <link name="arm_mount">
     <visual>
@@ -102,9 +102,12 @@
   </joint>
   <!-- ═══════════════════════════════════════════════
-       LEFT WHEEL
+       WHEELS
+       Z=0 relative to base_link because:
+       base_link center = wheel_r above ground
+       wheel axle = wheel_r above ground
+       therefore wheel axle Z offset from base_link = 0
        ═══════════════════════════════════════════════ -->
   <link name="left_wheel">
     <visual>
-      <origin xyz="0 0 0" rpy="0 0 0"/>
       <geometry>
         <cylinder radius="${wheel_r}" length="${wheel_t}"/>
@@ -115,5 +118,4 @@
     </visual>
     <collision>
-      <origin xyz="0 0 0" rpy="0 0 0"/>
       <geometry>
         <cylinder radius="${wheel_r}" length="${wheel_t}"/>
@@ -130,24 +132,21 @@
     </inertial>
   </link>
-  <joint name="left_wheel_joint" type="continuous">
-    <parent link="base_link"/>
-    <child  link="left_wheel"/>
+<joint name="left_wheel_joint" type="continuous">
+    <parent link="base_link"/>
+    <child link="left_wheel"/>
     <origin xyz="0 ${wheel_sep/2} ${-base_h/2+wheel_r}" rpy="${pi/2} 0 0"/>
-    <axis xyz="0 0 -1"/>
+    <axis xyz="0 1 0"/>
     <dynamics damping="0.1" friction="0.1"/>
   </joint>
-  <!-- ═══════════════════════════════════════════════
-       RIGHT WHEEL
-       ═══════════════════════════════════════════════ -->
   <link name="right_wheel">
     <visual>
-      <origin xyz="0 0 0" rpy="0 0 0"/>
       <geometry>
         <cylinder radius="${wheel_r}" length="${wheel_t}"/>
       </geometry>
-      <material name="tire_black"/>
-    </visual>
-    <collision>
-      <origin xyz="0 0 0" rpy="0 0 0"/>
+      <material name="tire_black">
+        <color rgba="0.1 0.1 0.1 1.0"/>
+      </material>
+    </visual>
+    <collision>
       <geometry>
         <cylinder radius="${wheel_r}" length="${wheel_t}"/>
@@ -164,13 +163,21 @@
     </inertial>
   </link>
-  <joint name="right_wheel_joint" type="continuous">
-    <parent link="base_link"/>
-    <child  link="right_wheel"/>
+<joint name="right_wheel_joint" type="continuous">
+    <parent link="base_link"/>
+    <child link="right_wheel"/>
     <origin xyz="0 ${-wheel_sep/2} ${-base_h/2+wheel_r}" rpy="${pi/2} 0 0"/>
-    <axis xyz="0 0 -1"/>
+    <axis xyz="0 1 0"/>
     <dynamics damping="0.1" friction="0.1"/>
   </joint>
   <!-- ═══════════════════════════════════════════════
-       CASTER WHEEL
+       CASTER
+       Z = -(base_h/2) drops to bottom of base_link
+       Then caster_r raises it so bottom touches ground
+       But base_link center is at wheel_r so:
+       caster bottom = wheel_r - base_h/2 + caster_r
+       This should equal 0 (ground level)
+       wheel_r=0.0425, base_h/2=0.065, caster_r=0.015
+       0.0425 - 0.065 + 0.015 = -0.0075 (slightly above)
+       Use -base_h/2 + caster_r to get close enough
        ═══════════════════════════════════════════════ -->
   <link name="caster_wheel">
@@ -195,9 +202,6 @@
     <parent link="base_link"/>
     <child  link="caster_wheel"/>
-    <origin xyz="${-(base_l/2-0.04)} 0 ${-base_h/2+caster_r}" rpy="0 0 0"/>
-  </joint>
-  <!-- ═══════════════════════════════════════════════
-       LIDAR LINK
-       ═══════════════════════════════════════════════ -->
+    <origin xyz="${-(base_l/2-0.04)} 0 ${-(base_h/2-caster_r)}" rpy="0 0 0"/>
+  </joint>
   <link name="lidar_link">
     <visual>
@@ -225,7 +229,4 @@
     <origin xyz="0.0 0.0 ${base_h/2+0.04}" rpy="0 0 0"/>
   </joint>
-  <!-- ═══════════════════════════════════════════════
-       IMU LINK
-       ═══════════════════════════════════════════════ -->
   <link name="imu_link">
     <inertial>
@@ -240,7 +241,4 @@
     <origin xyz="0 0 0" rpy="0 0 0"/>
   </joint>
-  <!-- ═══════════════════════════════════════════════
-       CAMERA LINK
-       ═══════════════════════════════════════════════ -->
   <link name="camera_link">
     <visual>
@@ -270,7 +268,4 @@
     <origin xyz="0 0 0" rpy="${-pi/2} 0 ${-pi/2}"/>
   </joint>
-  <!-- ═══════════════════════════════════════════════
-       GAZEBO CONTACT PROPERTIES
-       ═══════════════════════════════════════════════ -->
   <gazebo reference="caster_wheel">
     <mu1>0.0</mu1>
@@ -291,7 +286,4 @@
     <kd>100.0</kd>
   </gazebo>
-  <!-- ═══════════════════════════════════════════════
-       LIDAR SENSOR
-       ═══════════════════════════════════════════════ -->
   <gazebo reference="lidar_link">
     <sensor name="lidar" type="gpu_lidar">
@@ -323,27 +315,22 @@
     </sensor>
   </gazebo>
-  <!-- ═══════════════════════════════════════════════
-       DIFF DRIVE PLUGIN
-       child_frame_id = base_link (no base_footprint)
-       ═══════════════════════════════════════════════ -->
-  <gazebo>
-    <plugin filename="gz-sim-diff-drive-system"
-            name="gz::sim::systems::DiffDrive">
-      <left_joint>left_wheel_joint</left_joint>
-      <right_joint>right_wheel_joint</right_joint>
-      <wheel_separation>${wheel_sep}</wheel_separation>
-      <wheel_radius>${wheel_r}</wheel_radius>
-      <odom_publish_frequency>10</odom_publish_frequency>
-      <topic>cmd_vel</topic>
-      <odom_topic>odom</odom_topic>
-      <tf_topic>/tf</tf_topic>
-      <frame_id>odom</frame_id>
-      <child_frame_id>base_link</child_frame_id>
-      <max_linear_acceleration>1.0</max_linear_acceleration>
-    </plugin>
-    <plugin filename="gz-sim-joint-state-publisher-system"
-            name="gz::sim::systems::JointStatePublisher">
-      <topic>joint_states</topic>
-    </plugin>
-  </gazebo>
+<gazebo>
+  <plugin filename="gz-sim-diff-drive-system"
+          name="gz::sim::systems::DiffDrive">
+    <left_joint>left_wheel_joint</left_joint>
+    <right_joint>right_wheel_joint</right_joint>
+    <wheel_separation>${wheel_sep}</wheel_separation>
+    <wheel_radius>${wheel_r}</wheel_radius>
+    <topic>/cmd_vel</topic>
+    <odom_topic>odom</odom_topic>
+    <tf_topic>/tf</tf_topic>
+    <frame_id>odom</frame_id>
+    <child_frame_id>base_footprint</child_frame_id>
+    <odom_publish_frequency>30</odom_publish_frequency>
+    <max_linear_velocity>1.0</max_linear_velocity>
+    <max_angular_velocity>1.5</max_angular_velocity>
+    <max_linear_acceleration>1.0</max_linear_acceleration>
+    <max_angular_acceleration>1.5</max_angular_acceleration>
+  </plugin>
+</gazebo>
 </robot>

Commit message: refactor: update URDF robot model with dual casters and plugin-based joint publishing, and migrate to online_sync_launch for SLAM.

File: urdf/amr_robot.urdf.xacro (robot description, xacro)
@@ -135,6 +135,6 @@
     <parent link="base_link"/>
     <child link="left_wheel"/>
-    <origin xyz="0 ${wheel_sep/2} ${-base_h/2+wheel_r}" rpy="${pi/2} 0 0"/>
-    <axis xyz="0 1 0"/>
+    <origin xyz="0 ${wheel_sep/2} ${-base_h/2}" rpy="${pi/2} 0 0"/>
+    <axis xyz="0 0 -1"/>
     <dynamics damping="0.1" friction="0.1"/>
   </joint>
@@ -166,6 +166,6 @@
     <parent link="base_link"/>
     <child link="right_wheel"/>
-    <origin xyz="0 ${-wheel_sep/2} ${-base_h/2+wheel_r}" rpy="${pi/2} 0 0"/>
-    <axis xyz="0 1 0"/>
+    <origin xyz="0 ${-wheel_sep/2} ${-base_h/2}" rpy="${pi/2} 0 0"/>
+    <axis xyz="0 0 -1"/>
     <dynamics damping="0.1" friction="0.1"/>
   </joint>
@@ -181,5 +181,6 @@
        Use -base_h/2 + caster_r to get close enough
        ═══════════════════════════════════════════════ -->
-  <link name="caster_wheel">
+  <!-- REAR CASTER -->
+  <link name="rear_caster_wheel">
     <visual>
       <geometry><sphere radius="${caster_r}"/></geometry>
@@ -199,8 +200,32 @@
     </inertial>
   </link>
-  <joint name="caster_joint" type="fixed">
-    <parent link="base_link"/>
-    <child  link="caster_wheel"/>
-    <origin xyz="${-(base_l/2-0.04)} 0 ${-(base_h/2-caster_r)}" rpy="0 0 0"/>
+  <joint name="rear_caster_joint" type="fixed">
+    <parent link="base_link"/>
+    <child  link="rear_caster_wheel"/>
+    <origin xyz="${-(base_l/2-0.04)} 0 ${-base_h/2 - wheel_r + caster_r}" rpy="0 0 0"/>
+  </joint>
+  <!-- FRONT CASTER -->
+  <link name="front_caster_wheel">
+    <visual>
+      <geometry><sphere radius="${caster_r}"/></geometry>
+      <material name="light_gray">
+        <color rgba="0.6 0.6 0.6 1.0"/>
+      </material>
+    </visual>
+    <collision>
+      <geometry><sphere radius="${caster_r}"/></geometry>
+    </collision>
+    <inertial>
+      <mass value="0.05"/>
+      <inertia
+        ixx="0.000025" ixy="0" ixz="0"
+        iyy="0.000025" iyz="0"
+        izz="0.000025"/>
+    </inertial>
+  </link>
+  <joint name="front_caster_joint" type="fixed">
+    <parent link="base_link"/>
+    <child  link="front_caster_wheel"/>
+    <origin xyz="${(base_l/2-0.04)} 0 ${-base_h/2 - wheel_r + caster_r}" rpy="0 0 0"/>
   </joint>
   <link name="lidar_link">
@@ -268,5 +293,11 @@
     <origin xyz="0 0 0" rpy="${-pi/2} 0 ${-pi/2}"/>
   </joint>
-  <gazebo reference="caster_wheel">
+  <gazebo reference="rear_caster_wheel">
+    <mu1>0.0</mu1>
+    <mu2>0.0</mu2>
+    <kp>1000000.0</kp>
+    <kd>100.0</kd>
+  </gazebo>
+  <gazebo reference="front_caster_wheel">
     <mu1>0.0</mu1>
     <mu2>0.0</mu2>
@@ -333,4 +364,10 @@
     <max_angular_acceleration>1.5</max_angular_acceleration>
   </plugin>
+  <plugin filename="gz-sim-joint-state-publisher-system"
+          name="gz::sim::systems::JointStatePublisher">
+    <topic>joint_states</topic>
+    <joint_name>left_wheel_joint</joint_name>
+    <joint_name>right_wheel_joint</joint_name>
+  </plugin>
 </gazebo>
 </robot>

Commit message: feat: add QR code station models, integrate camera sensor, and update gazebo launch with coordinate overrides

File: urdf/amr_robot.urdf.xacro (robot description, xacro)
@@ -286,5 +286,5 @@
     <parent link="base_link"/>
     <child  link="camera_link"/>
-    <origin xyz="${base_l/2-0.01} 0 ${base_h/2-0.01}" rpy="0 0 0"/>
+    <origin xyz="${base_l/2-0.01} 0 ${base_h/2-0.01}" rpy="0 0.2618 0"/>
   </joint>
   <joint name="camera_optical_joint" type="fixed">
@@ -293,4 +293,25 @@
     <origin xyz="0 0 0" rpy="${-pi/2} 0 ${-pi/2}"/>
   </joint>
+  <gazebo reference="camera_link">
+    <sensor name="camera" type="camera">
+      <always_on>true</always_on>
+      <visualize>true</visualize>
+      <update_rate>30</update_rate>
+      <topic>/camera/image_raw</topic>
+      <gz_frame_id>camera_optical_frame</gz_frame_id>
+      <camera>
+        <horizontal_fov>1.047</horizontal_fov>
+        <image>
+          <width>640</width>
+          <height>480</height>
+          <format>R8G8B8</format>
+        </image>
+        <clip>
+          <near>0.1</near>
+          <far>10.0</far>
+        </clip>
+      </camera>
+    </sensor>
+  </gazebo>
   <gazebo reference="rear_caster_wheel">
     <mu1>0.0</mu1>

Commit message: feat: implement mission management, inventory logging, and update QR detection and station models

File: urdf/amr_robot.urdf.xacro (robot description, xacro)
@@ -286,5 +286,5 @@
     <parent link="base_link"/>
     <child  link="camera_link"/>
-    <origin xyz="${base_l/2-0.01} 0 ${base_h/2-0.01}" rpy="0 0.2618 0"/>
+    <origin xyz="${base_l/2-0.01} 0 0.1925" rpy="0 0.2618 0"/>
   </joint>
   <joint name="camera_optical_joint" type="fixed">
@@ -391,4 +391,14 @@
     <joint_name>right_wheel_joint</joint_name>
   </plugin>
+  <plugin filename="gz-sim-pose-publisher-system"
+          name="gz::sim::systems::PosePublisher">
+    <publish_link_pose>false</publish_link_pose>
+    <publish_collision_pose>false</publish_collision_pose>
+    <publish_visual_pose>false</publish_visual_pose>
+    <publish_nested_model_pose>false</publish_nested_model_pose>
+    <publish_model_pose>true</publish_model_pose>
+    <use_pose_vector_msg>false</use_pose_vector_msg>
+    <update_rate>50.0</update_rate>
+  </plugin>
 </gazebo>
 </robot>
